File: electrical-design/dmats_hw_v2_0/portenta_h7.kicad_sch (KiCad schematic)
At the start: 1 part, among them U5 ABX00042

Commit message: bulk of PCB design layout complete
Parts:
- removed U5: ABX00042, DMATS_capstone:MODULE_ABX00042, symbol DMATS_capstone:ABX00042
